File: memory-display.kicad_pcb (KiCad board)
At the start: 2 copper layers, 1 part, among them J1 TEENSY LC

Commit message: finished schematic and start layout
Parts:
- added CAP1: CAP15, Wickerlib:CAPSENSE-CIRCLE-D10MM, F.Cu at (128.5, 121.5)
- added J2: SHARP-MEM-DISP, Wickerlib:CONN-HEADER-STRAIGHT-P2.54MM-1x09, F.Cu at (131.8, 82.2)
- added J3: I2C-BMP180, Wickerlib:CONN-HEADER-STRAIGHT-P2.54MM-1x07, F.Cu at (72.0, 83.0)
- added P1: D0, Wickerlib:CONN-HEADER-STRAIGHT-P2.54MM-1x01, F.Cu at (87.0, 75.2)
- added P10: D9, Wickerlib:CONN-HEADER-STRAIGHT-P2.54MM-1x01, F.Cu at (84.8, 97.8)
- added P11: D12, Wickerlib:CONN-HEADER-STRAIGHT-P2.54MM-1x01, F.Cu at (86.0, 107.2)
- added P12: D14, Wickerlib:CONN-HEADER-STRAIGHT-P2.54MM-1x01, F.Cu at (118.8, 103.2)
- added P13: D16, Wickerlib:CONN-HEADER-STRAIGHT-P2.54MM-1x01, F.Cu at (118.0, 97.6)
- added P14: D17, Wickerlib:CONN-HEADER-STRAIGHT-P2.54MM-1x01, F.Cu at (118.2, 91.6)
- added P15: D20, Wickerlib:CONN-HEADER-STRAIGHT-P2.54MM-1x01, F.Cu at (118.0, 86.0)
- added P16: D21, Wickerlib:CONN-HEADER-STRAIGHT-P2.54MM-1x01, F.Cu at (118.6, 78.8)
- added P17: D22, Wickerlib:CONN-HEADER-STRAIGHT-P2.54MM-1x01, F.Cu at (124.4, 80.8)
- added P18: D23, Wickerlib:CONN-HEADER-STRAIGHT-P2.54MM-1x01, F.Cu at (124.8, 76.8)
- added P19: 17A, Wickerlib:CONN-HEADER-STRAIGHT-P2.54MM-1x01, F.Cu at (98.6, 118.4)
- added P2: D1, Wickerlib:CONN-HEADER-STRAIGHT-P2.54MM-1x01, F.Cu at (87.0, 79.0)
- added P20: DAC, Wickerlib:CONN-HEADER-STRAIGHT-P2.54MM-1x01, F.Cu at (109.0, 118.4)
- added P21: PGM, Wickerlib:CONN-HEADER-STRAIGHT-P2.54MM-1x01, F.Cu at (106.8, 124.2)
- added P22: PGM, Wickerlib:CONN-HEADER-STRAIGHT-P2.54MM-1x01, F.Cu at (103.0, 117.6)
- added P23: 3v3, Wickerlib:CONN-HEADER-STRAIGHT-P2.54MM-1x01, F.Cu at (117.6, 67.8)
- added P24: CS, Wickerlib:CONN-HEADER-STRAIGHT-P2.54MM-1x01, F.Cu at (118.2, 113.2)
- added P25: DI, Wickerlib:CONN-HEADER-STRAIGHT-P2.54MM-1x01, F.Cu at (90.6, 119.0)
- added P26: CLK, Wickerlib:CONN-HEADER-STRAIGHT-P2.54MM-1x01, F.Cu at (89.4, 102.0)
- added P3: D2, Wickerlib:CONN-HEADER-STRAIGHT-P2.54MM-1x01, F.Cu at (87.0, 83.2)
- added P4: D3, Wickerlib:CONN-HEADER-STRAIGHT-P2.54MM-1x01, F.Cu at (91.8, 84.0)
- added P5: D4, Wickerlib:CONN-HEADER-STRAIGHT-P2.54MM-1x01, F.Cu at (84.5, 90.5)
- added P6: D5, Wickerlib:CONN-HEADER-STRAIGHT-P2.54MM-1x01, F.Cu at (92.5, 87.2)
- added P7: D6, Wickerlib:CONN-HEADER-STRAIGHT-P2.54MM-1x01, F.Cu at (89.5, 90.5)
- added P8: D7, Wickerlib:CONN-HEADER-STRAIGHT-P2.54MM-1x01, F.Cu at (91.5, 94.8)
- added P9: D8, Wickerlib:CONN-HEADER-STRAIGHT-P2.54MM-1x01, F.Cu at (78.4, 94.4)
- J1: value TEENSY LC -> TEENSY-LC
Connections:
- J1 pad 0: (no net) -> /D0
- J1 pad 1: (no net) -> /D1
- J1 pad 10: (no net) -> /CLK
- J1 pad 11: (no net) -> /D11
- J1 pad 12: (no net) -> /D12
- J1 pad 13: (no net) -> /CS
- J1 pad 14: (no net) -> /D14
- J1 pad 15: (no net) -> /D15
- J1 pad 16: (no net) -> /D16
- J1 pad 17: (no net) -> /D17
- J1 pad 17A: (no net) -> /D17(VIN)
- J1 pad 18: (no net) -> /D18
- J1 pad 19: (no net) -> /D19
- J1 pad 2: (no net) -> /D2
- J1 pad 20: (no net) -> /D20
- J1 pad 21: (no net) -> /D21
- J1 pad 22: (no net) -> /D22
- J1 pad 23: (no net) -> /D23
- J1 pad 3: (no net) -> /D3
- J1 pad 4: (no net) -> /D4
- J1 pad 5: (no net) -> /D5
- J1 pad 6: (no net) -> /D6
- J1 pad 7: (no net) -> /D7
- J1 pad 8: (no net) -> /D8
- J1 pad 9: (no net) -> /D9
- J1 pad DAC: (no net) -> /DAC
- J1 pad PGM: (no net) -> /PROG
- J1 pad VIN: (no net) -> +3V3

Commit message: finish layout
Parts:
- removed J2: SHARP-MEM-DISP, Wickerlib:CONN-HEADER-STRAIGHT-P2.54MM-1x09
- removed J3: I2C-BMP180, Wickerlib:CONN-HEADER-STRAIGHT-P2.54MM-1x07
- added G***: LOGO, teensy-big-oled:osh-park-logo-200dpi-norm-silk, F.Cu at (95.4, 122.8)
- added I2C-BMP180: I2C-BMP180, Wickerlib:Pin_Header_Straight_1x07, F.Cu at (125.3, 126.3)
- added REF**: Symbol_OSHW-Logo_SilkScreen, Symbols:Symbol_OSHW-Logo_SilkScreen, B.Cu at (95.7, 121.4)
- added SHARP Memory Display: SHARP-MEM-DISP, Wickerlib:Pin_Header_Straight_1x09, F.Cu at (103.0, 83.8)
- moved 3V3 54.0 mm to (133.1, 119.5), turned to 270 degrees
- moved D0 49.1 mm to (133.0, 92.3), turned to 270 degrees
- moved D1 44.5 mm to (129.5, 92.3), turned to 270 degrees
- moved D23 43.0 mm to (129.6, 119.5), turned to 270 degrees
- moved D21 41.4 mm to (126.1, 119.5), turned to 270 degrees
- moved D2 39.9 mm to (125.9, 92.3), turned to 270 degrees
- moved D22 38.8 mm to (122.6, 119.5), turned to 270 degrees
- moved D4 34.3 mm to (118.8, 92.3), turned to 270 degrees
- moved D20 33.5 mm to (119.1, 119.5), turned to 270 degrees
- moved CAP15 33.0 mm to (95.5, 122.6), turned to 270 degrees
- moved D3 31.7 mm to (122.4, 92.3), turned to 270 degrees
- moved J1 30.9 mm to (123.1, 108.1), turned to 270 degrees
- moved D17 28.1 mm to (115.6, 119.5), turned to 270 degrees
- moved DI 27.0 mm to (93.9, 92.3), turned to 270 degrees
- moved D8 26.3 mm to (104.6, 92.3), turned to 270 degrees
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- renumbered P19 to 17A, P23 to 3V3, CAP1 to CAP15, P26 to CLK, P24 to CS, P1 to D0, P2 to D1, P11 to D12, P12 to D14, P13 to D16, P14 to D17, P3 to D2, P15 to D20, P16 to D21, P17 to D22, P18 to D23, P4 to D3, P5 to D4, P6 to D5, P7 to D6, P8 to D7, P9 to D8, P10 to D9, P20 to DAC, P25 to DI, P22 to GND, P21 to PGM
Routing:
- net +3V3: track 0.00 -> 93.0 mm, vias 0 -> 3
- net /CS: track 0.00 -> 45.7 mm, vias 0 -> 1
- net /D11: track 0.00 -> 30.1 mm
- net /CLK: track 0.00 -> 29.1 mm, vias 0 -> 2
- net /D19: track 0.00 -> 14.0 mm
- net /D15: track 0.00 -> 13.9 mm, vias 0 -> 1
- net /D18: track 0.00 -> 13.9 mm
- net /D9: track 0.00 -> 9.42 mm
- net /D14: track 0.00 -> 8.68 mm
- net /D21: track 0.00 -> 8.61 mm, vias 0 -> 1
- net /DAC: track 0.00 -> 8.54 mm
- net /D17: track 0.00 -> 8.44 mm, vias 0 -> 1
- net /D8: track 0.00 -> 8.41 mm
- net /D17(VIN): track 0.00 -> 8.39 mm
- net /PROG: track 0.00 -> 8.18 mm
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- added copper zone on B.Cu, net GND
Other:
- board outline added: 48.9 x 50.8 mm
- net class Default: via_dia 0.6858 -> 0.7874; via_drill 0.3302 -> 0.5334
- rule trace_min: 0.1524 -> 0.254
- rule via_min_drill: 0.3302 -> 0.508
- rule via_min_size: 0.6858 -> 0.762
- board text added: "Drew Fustini <drew@oshpark.com>"
- board text added: "SHARP Memory Display + Teensy LC https://github.com/pdp7/memory-display by Drew Fustini <drew@oshpark.com>"
- board text removed: "17(VIN) 3.3V GND PROG DAC"
- board text removed: "GND 0 1 2 3 4 5 6 7 8 9 10 11 12"
- board text removed: "Note: Please feel free to delete the silk. It is not a part of the footprint. (Also feel free to delete this note.)"
- board text removed: "VIN GND 3.3V 23 22 21 20 19 18 17 16 15 14 13"
