File: memory-display.sch (KiCad schematic (older format))
At the start: 1 part, among them J1 TEENSY-LC

Commit message: finished schematic and start layout
Parts:
- added CAP1: CAP15, Wickerlib:CAPSENSE-CIRCLE-D10MM, symbol CAPSENSE_CIRCLE
- added J2: SHARP-MEM-DISP, Wickerlib:CONN-HEADER-STRAIGHT-P2.54MM-1x09, symbol HEADER-MALE-9POS-TH-1x09-P0.1IN
- added J3: I2C-BMP180, Wickerlib:CONN-HEADER-STRAIGHT-P2.54MM-1x07, symbol HEADER-MALE-7POS-TH-1x07-P0.1IN
- added P1: D0, Wickerlib:CONN-HEADER-STRAIGHT-P2.54MM-1x01, symbol HEADER-MALE-1POS-TH-1x01
- added P10: D9, Wickerlib:CONN-HEADER-STRAIGHT-P2.54MM-1x01, symbol HEADER-MALE-1POS-TH-1x01
- added P11: D12, Wickerlib:CONN-HEADER-STRAIGHT-P2.54MM-1x01, symbol HEADER-MALE-1POS-TH-1x01
- added P12: D14, Wickerlib:CONN-HEADER-STRAIGHT-P2.54MM-1x01, symbol HEADER-MALE-1POS-TH-1x01
- added P13: D16, Wickerlib:CONN-HEADER-STRAIGHT-P2.54MM-1x01, symbol HEADER-MALE-1POS-TH-1x01
- added P14: D17, Wickerlib:CONN-HEADER-STRAIGHT-P2.54MM-1x01, symbol HEADER-MALE-1POS-TH-1x01
- added P15: D20, Wickerlib:CONN-HEADER-STRAIGHT-P2.54MM-1x01, symbol HEADER-MALE-1POS-TH-1x01
- added P16: D21, Wickerlib:CONN-HEADER-STRAIGHT-P2.54MM-1x01, symbol HEADER-MALE-1POS-TH-1x01
- added P17: D22, Wickerlib:CONN-HEADER-STRAIGHT-P2.54MM-1x01, symbol HEADER-MALE-1POS-TH-1x01
- added P18: D23, Wickerlib:CONN-HEADER-STRAIGHT-P2.54MM-1x01, symbol HEADER-MALE-1POS-TH-1x01
- added P19: 17A, Wickerlib:CONN-HEADER-STRAIGHT-P2.54MM-1x01, symbol HEADER-MALE-1POS-TH-1x01
- added P2: D1, Wickerlib:CONN-HEADER-STRAIGHT-P2.54MM-1x01, symbol HEADER-MALE-1POS-TH-1x01
- added P20: DAC, Wickerlib:CONN-HEADER-STRAIGHT-P2.54MM-1x01, symbol HEADER-MALE-1POS-TH-1x01
- added P21, P22: PGM, Wickerlib:CONN-HEADER-STRAIGHT-P2.54MM-1x01, symbol HEADER-MALE-1POS-TH-1x01
- added P23: 3v3, Wickerlib:CONN-HEADER-STRAIGHT-P2.54MM-1x01, symbol HEADER-MALE-1POS-TH-1x01
- added P24: CS, Wickerlib:CONN-HEADER-STRAIGHT-P2.54MM-1x01, symbol HEADER-MALE-1POS-TH-1x01
- added P25: DI, Wickerlib:CONN-HEADER-STRAIGHT-P2.54MM-1x01, symbol HEADER-MALE-1POS-TH-1x01
- added P26: CLK, Wickerlib:CONN-HEADER-STRAIGHT-P2.54MM-1x01, symbol HEADER-MALE-1POS-TH-1x01
- added P3: D2, Wickerlib:CONN-HEADER-STRAIGHT-P2.54MM-1x01, symbol HEADER-MALE-1POS-TH-1x01
- added P4: D3, Wickerlib:CONN-HEADER-STRAIGHT-P2.54MM-1x01, symbol HEADER-MALE-1POS-TH-1x01
- added P5: D4, Wickerlib:CONN-HEADER-STRAIGHT-P2.54MM-1x01, symbol HEADER-MALE-1POS-TH-1x01
- added P6: D5, Wickerlib:CONN-HEADER-STRAIGHT-P2.54MM-1x01, symbol HEADER-MALE-1POS-TH-1x01
- added P7: D6, Wickerlib:CONN-HEADER-STRAIGHT-P2.54MM-1x01, symbol HEADER-MALE-1POS-TH-1x01
- added P8: D7, Wickerlib:CONN-HEADER-STRAIGHT-P2.54MM-1x01, symbol HEADER-MALE-1POS-TH-1x01
- added P9: D8, Wickerlib:CONN-HEADER-STRAIGHT-P2.54MM-1x01, symbol HEADER-MALE-1POS-TH-1x01
Connections:
- net labels added: 3V3, 3VO, CLK, CS, DI, DISP, EIN, EMO, SCK, SCL, SDA, SDI, SDO
- wire segments 36 -> 73
- no-connect marks 0 -> 7

Commit message: finish layout
Parts:
- I2C-BMP180: renamed from J3; footprint Wickerlib:CONN-HEADER-STRAIGHT-P2.54MM-1x07 -> Wickerlib:Pin_Header_Straight_1x07
- J1: footprint TEENSY-LC -> Wickerlib:TEENSY-LC
- SHARP-MEM-DISP1: renamed from J2; footprint Wickerlib:CONN-HEADER-STRAIGHT-P2.54MM-1x09 -> Wickerlib:Pin_Header_Straight_1x09
Changed lines of the file:
@@
 LIBS:Symbols_DCDC-ACDC-Converter_RevC_20Jul2012
 LIBS:SymbolsSimilarEN60617+oldDIN617-RevE8
-LIBS:wickerlib
-LIBS:chip-dips
 LIBS:memory-display-cache
 EELAYER 25 0
@@
 F 0 "J1" H 2575 4450 50  0000 L CNN
 F 1 "TEENSY-LC" H 2575 4350 50  0000 L CNN
-F 2 "TEENSY-LC" V 2525 2800 50  0001 C CIN
+F 2 "Wickerlib:TEENSY-LC" V 2525 2800 50  0001 C CIN
 F 3 "https://cdn.harwin.com/pdfs/60page140.pdf" H 2825 3200 5   0001 C CNN
 F 4 "TEENSY-LC" V 2525 2800 50  0001 C CIN "Package"
@@
 $EndComp
 $Comp
-L HEADER-MALE-9POS-TH-1x09-P0.1IN J2
+L HEADER-MALE-9POS-TH-1x09-P0.1IN SHARP-MEM-DISP1
 U 1 1 57959F85
 P 5700 3250
-F 0 "J2" H 5682 3746 50  0000 L CNN
-F 1 "SHARP-MEM-DISP" H 5950 3500 50  0000 L CNN
-F 2 "Wickerlib:CONN-HEADER-STRAIGHT-P2.54MM-1x09" H 5700 2900 50  0001 C CIN
+F 0 "SHARP-MEM-DISP1" V 5925 2950 50  0000 L CNN
+F 1 "SHARP-MEM-DISP" H 5950 3500 50  0001 L CNN
+F 2 "Wickerlib:Pin_Header_Straight_1x09" H 5700 2900 50  0001 C CIN
 F 3 "https://cdn.harwin.com/pdfs/60page140.pdf" H 5700 3250 5   0001 C CNN
 F 4 "Pin_Header_Straight_1x09" H 5700 2900 50  0001 C CIN "Package"
@@
 SDA
 $Comp
-L HEADER-MALE-7POS-TH-1x07-P0.1IN J3
+L HEADER-MALE-7POS-TH-1x07-P0.1IN I2C-BMP180
 U 1 1 5795B6CB
 P 7175 4950
-F 0 "J3" H 7175 5400 50  0000 L CNN
-F 1 "I2C-BMP180" V 7325 4750 50  0000 L CNN
-F 2 "Wickerlib:CONN-HEADER-STRAIGHT-P2.54MM-1x07" H 7175 4600 50  0001 C CIN
+F 0 "I2C-BMP180" V 7350 4750 50  0000 L CNN
+F 1 "I2C-BMP180" V 7325 4750 50  0001 L CNN
+F 2 "Wickerlib:Pin_Header_Straight_1x07" H 7175 4600 50  0001 C CIN
 F 3 "https://cdn.harwin.com/pdfs/60page140.pdf" H 7175 4950 5   0001 C CNN
 F 4 "Pin_Header_Straight_1x07" H 7175 4600 50  0001 C CIN "Package"
